File: drum_trigger.kicad_sch (KiCad schematic)
At the start: 6 parts, among them J1 528520870, J2 528520870, J3 528520870

Commit message: Production ready pcb
Parts:
- J1, J2, J3: now left out of the parts list
Changed lines of the file:
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@@
+			)
+		)
+		(property "LTSC" ""
+			(at 74.93 40.64 0)
+			(effects
+				(font
+					(size 1.27 1.27)
+				)
+				(hide yes)
 			)
 		)
@@
 			)
 		)
+		(property "LTSC" ""
+			(at 92.71 45.72 0)
+			(effects
+				(font
+					(size 1.27 1.27)
+				)
+				(hide yes)
+			)
+		)
 		(pin "2"
 		)
@@
 		(unit 1)
 		(exclude_from_sim yes)
-		(in_bom yes)
+		(in_bom no)
 		(on_board yes)
 		(dnp no)
@@
 		(unit 1)
 		(exclude_from_sim yes)
-		(in_bom yes)
+		(in_bom no)
 		(on_board no)
 		(dnp no)
@@
 		)
 		(property "STANDARD" ""
+			(at 31.75 45.72 0)
+			(effects
+				(font
+					(size 1.27 1.27)
+				)
+				(hide yes)
+			)
+		)
+		(property "LTSC" ""
 			(at 31.75 45.72 0)
 			(effects
@@
 		(unit 1)
 		(exclude_from_sim yes)
-		(in_bom yes)
+		(in_bom no)
 		(on_board no)
 		(dnp no)
@@
 		)
 		(property "STANDARD" ""
+			(at 34.29 97.79 0)
+			(effects
+				(font
+					(size 1.27 1.27)
+				)
+				(hide yes)
+			)
+		)
+		(property "LTSC" ""
 			(at 34.29 97.79 0)
 			(effects
@@
 			)
 		)
+		(property "LTSC" ""
+			(at 74.93 50.8 0)
+			(effects
+				(font
+					(size 1.27 1.27)
+				)
+				(hide yes)
+			)
+		)
 		(pin "1"
 		)
@@
 		(unit 1)
 		(exclude_from_sim yes)
-		(in_bom yes)
+		(in_bom no)
 		(on_board no)
 		(dnp no)
@@
 			)
 		)
+		(property "LTSC" ""
+			(at 67.31 97.79 0)
+			(effects
+				(font
+					(size 1.27 1.27)
+				)
+				(hide yes)
+			)
+		)
 		(pin "6"
 		)
@@
 	)
 	(sheet
-		(at 132.08 60.96)
+		(at 245.11 119.38)
 		(size 34.29 19.05)
-		(exclude_from_sim no)
-		(in_bom yes)
+		(exclude_from_sim yes)
+		(in_bom no)
 		(on_board no)
 		(dnp yes)
@@
 		)
 		(property "Sheetname" "TriggerPairLM324"
-			(at 132.08 60.2484 0)
+			(at 245.11 118.6684 0)
 			(effects
 				(font
@@
 		)
 		(property "Sheetfile" "trigger_pair_lm324.kicad_sch"
-			(at 132.08 80.5946 0)
-			(effects
-				(font
+			(at 245.11 139.0146 0)
+			(effects
+				(font

Commit message: Simulation fixes + board fixes
Other:
- removed sheet TriggerPairLM324
- sheet TrigEn ports: added +3V3IN, TRIG_A_EN, TRIG_A_IN, TRIG_B_EN, TRIG_B_IN; removed none
- sheet TriggerPair ports: added none; removed TRIG_A_EN, TRIG_B_EN
- moved on the sheet: V1, V2, V3

Commit message: Add channels
Parts:
- added D1: KT-0805G, LED_SMD:LED_0805_2012Metric, symbol Device:LED
- added H1, H2, H3, H4: MountingHole_Pad, MountingHole:MountingHole_2.2mm_M2_Pad_Via, symbol Mechanical:MountingHole_Pad
- added J1: Conn_01x03_Pin, Connector_JST:JST_PH_B3B-PH-K_1x03_P2.00mm_Vertical, symbol Connector:Conn_01x03_Pin
- added J3: Conn_01x10, Connector_JST:JST_ZH_B10B-ZR_1x10_P1.50mm_Vertical, symbol Connector_Generic:Conn_01x10
- added R1: 4.7k, Resistor_SMD:R_0603_1608Metric, symbol Device:R_Small
- added R104, R105, R106, R107, R108, R109, R110, R111: 100, R_0402_custom:R_0402_1005Metric, symbol Device:R_Small
- renumbered J1 to J2, J2 to J4, J3 to J5
Connections:
- net +9V: now also J1.1 (Pin_1), R1.1
- net -9V: now also J1.3 (Pin_3)
- net GND: now also D1.1 (K), H1.1, H2.1, H3.1, H4.1, J1.2 (Pin_2), J3.1 (Pin_1), J3.10 (Pin_10)
- net TRIG_T1: now also R106.1
- net TRIG_T2: now also R109.1
- net TRIG_T3: now also R104.1
- net TRIG_T4: now also R111.1
- net TRIG_T5: now also R108.1
- net TRIG_T6: now also R107.1
- net TRIG_T7: now also R110.1
- net TRIG_T8: now also R105.1
- new net: J3.9 (Pin_9), R111.2
- new net: J3.2 (Pin_2), R104.2
- new net: J3.3 (Pin_3), R105.2
- new net: J3.4 (Pin_4), R106.2
- new net: J3.5 (Pin_5), R107.2
- new net: J3.6 (Pin_6), R108.2
- new net: J3.7 (Pin_7), R109.2
- new net: J3.8 (Pin_8), R110.2
- new net: D1.2 (A), R1.2
Other:
- added sheet TriggerPair1 (trigger_pair.kicad_sch)
- added sheet TriggerPair2 (trigger_pair.kicad_sch)
- added sheet TriggerPair3 (trigger_pair.kicad_sch)
- note added: ".tran 1u 60m"
- moved on the sheet: V1, V2, V3
