File: trig_en.kicad_sch (KiCad schematic)
At the start: 14 parts, among them U10 1SS362FV_L3F, U8 1SS362FV_L3F, U9 SN74HC14DR

Commit message: Double trigger layout to test
Parts:
- renumbered C15 to C16, C16 to C17, C17 to C18, C18 to C19, C19 to C20, U8 to U2, U9 to U3, U10 to U4

Commit message: Simulation fixes + board fixes
Parts:
- removed U2, U4: 1SS362FV_L3F, mod:DIODE_1SS362FV, symbol DIODE_SET_1SS362FV:1SS362FV_L3F
- added D8, D9: BAV99,215, Package_TO_SOT_SMD:SOT-23, symbol Diode:BAV99
Connections:
- net +3V3IN is gone; now on net +3V3: C20.1, U3.14 (VCC)
- net +3V3: now also D8.2 (A), D9.2 (A)
- net CH1_SIG_TO_DETECTOR: now also D8.3 (K)
- net CH2_SIG_TO_DETECTOR: now also D9.3 (K)
- net GND: now also D8.1 (K), D9.1 (K)

Commit message: Add channels
Parts:
- renumbered C16 to C17, C17 to C18, C18 to C19, C19 to C20, C20 to C21, U3 to U2
Changed lines of the file:
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@@
 		(dnp no)
 		(fields_autoplaced yes)
-		(property "Reference" "#PWR047"
+		(property "Reference" "#PWR046"
 			(at 148.59 172.72 0)
 			(effects
@@
 			(project "drum_trigger"
 				(path "/5aab9db2-4b7f-4c4d-b6d6-4c2a1995e627/7d7842c4-e5e3-46ac-bf06-c89ddb20aca8"
-					(reference "#PWR047")
+					(reference "#PWR046")
 					(unit 1)
 				)
@@
 		(on_board yes)
 		(dnp no)
-		(property "Reference" "#PWR036"
+		(property "Reference" "#PWR039"
 			(at 133.35 50.8 0)
 			(effects
@@
 			(project "drum_trigger"
 				(path "/5aab9db2-4b7f-4c4d-b6d6-4c2a1995e627/7d7842c4-e5e3-46ac-bf06-c89ddb20aca8"
-					(reference "#PWR036")
+					(reference "#PWR039")
 					(unit 1)
 				)
@@
 		(dnp no)
 		(fields_autoplaced yes)
-		(property "Reference" "C20"
+		(property "Reference" "C21"
 			(at 168.91 148.5962 0)
 			(effects
@@
 			(project "drum_trigger"
 				(path "/5aab9db2-4b7f-4c4d-b6d6-4c2a1995e627/7d7842c4-e5e3-46ac-bf06-c89ddb20aca8"
-					(reference "C20")
+					(reference "C21")
 					(unit 1)
 				)
@@
 		(dnp no)
 		(fields_autoplaced yes)
-		(property "Reference" "#PWR039"
+		(property "Reference" "#PWR041"
 			(at 146.05 73.66 0)
 			(effects
@@
 			(project "drum_trigger"
 				(path "/5aab9db2-4b7f-4c4d-b6d6-4c2a1995e627/7d7842c4-e5e3-46ac-bf06-c89ddb20aca8"
-					(reference "#PWR039")
+					(reference "#PWR041")
 					(unit 1)
 				)
@@
 		(on_board yes)
 		(dnp no)
-		(property "Reference" "C17"
+		(property "Reference" "C18"
 			(at 178.816 57.912 90)
 			(effects
@@
 			(project "drum_trigger"
 				(path "/5aab9db2-4b7f-4c4d-b6d6-4c2a1995e627/7d7842c4-e5e3-46ac-bf06-c89ddb20aca8"
-					(reference "C17")
+					(reference "C18")
 					(unit 1)
 				)
@@
 		(dnp no)
 		(fields_autoplaced yes)
-		(property "Reference" "#PWR045"
+		(property "Reference" "#PWR044"
 			(at 142.24 118.11 0)
 			(effects
@@
 			(project "drum_trigger"
 				(path "/5aab9db2-4b7f-4c4d-b6d6-4c2a1995e627/7d7842c4-e5e3-46ac-bf06-c89ddb20aca8"
-					(reference "#PWR045")
+					(reference "#PWR044")
 					(unit 1)
 				)
@@
 		(dnp no)
 		(fields_autoplaced yes)
-		(property "Reference" "U3"
+		(property "Reference" "U2"
 			(at 163.83 90.17 0)
 			(effects
@@
 			(project "drum_trigger"
 				(path "/5aab9db2-4b7f-4c4d-b6d6-4c2a1995e627/7d7842c4-e5e3-46ac-bf06-c89ddb20aca8"
-					(reference "U3")
+					(reference "U2")
 					(unit 2)
 				)
@@
 		(on_board yes)
 		(dnp no)
-		(property "Reference" "C18"
+		(property "Reference" "C19"
 			(at 140.716 102.362 90)
 			(effects
@@
 			(project "drum_trigger"
 				(path "/5aab9db2-4b7f-4c4d-b6d6-4c2a1995e627/7d7842c4-e5e3-46ac-bf06-c89ddb20aca8"
-					(reference "C18")
+					(reference "C19")
 					(unit 1)
 				)
@@
 		(dnp no)
 		(fields_autoplaced yes)
-		(property "Reference" "#PWR038"
+		(property "Reference" "#PWR040"
 			(at 120.65 52.07 0)
 			(effects
@@
 			(project "drum_trigger"
 				(path "/5aab9db2-4b7f-4c4d-b6d6-4c2a1995e627/7d7842c4-e5e3-46ac-bf06-c89ddb20aca8"
-					(reference "#PWR038")
+					(reference "#PWR040")
 					(unit 1)
 				)
@@
 		(dnp no)
 		(fields_autoplaced yes)
-		(property "Reference" "#PWR046"
+		(property "Reference" "#PWR045"
 			(at 180.34 118.11 0)
 			(effects
@@
 			(project "drum_trigger"
 				(path "/5aab9db2-4b7f-4c4d-b6d6-4c2a1995e627/7d7842c4-e5e3-46ac-bf06-c89ddb20aca8"
-					(reference "#PWR046")
+					(reference "#PWR045")
 					(unit 1)
 				)
@@
 		(dnp no)
 		(fields_autoplaced yes)
-		(property "Reference" "#PWR049"
+		(property "Reference" "#PWR038"
 			(at 110.49 29.21 0)
 			(effects
@@
 			(project "drum_trigger"
 				(path "/5aab9db2-4b7f-4c4d-b6d6-4c2a1995e627/7d7842c4-e5e3-46ac-bf06-c89ddb20aca8"
-					(reference "#PWR049")
+					(reference "#PWR038")
 					(unit 1)
 				)
@@
 		(dnp no)
 		(fields_autoplaced yes)
-		(property "Reference" "#PWR042"
+		(property "Reference" "#PWR043"
 			(at 133.35 95.25 0)
 			(effects
@@
 			(project "drum_trigger"
 				(path "/5aab9db2-4b7f-4c4d-b6d6-4c2a1995e627/7d7842c4-e5e3-46ac-bf06-c89ddb20aca8"
-					(reference "#PWR042")
+					(reference "#PWR043")
 					(unit 1)
 				)
@@
 		(dnp no)
 		(fields_autoplaced yes)
-		(property "Reference" "U3"
+		(property "Reference" "U2"
 			(at 154.94 149.8599 0)
 			(effects
@@
 			(project "drum_trigger"
 				(path "/5aab9db2-4b7f-4c4d-b6d6-4c2a1995e627/7d7842c4-e5e3-46ac-bf06-c89ddb20aca8"
-					(reference "U3")
+					(reference "U2")
 					(unit 7)
 				)
@@
 		(dnp no)
 		(fields_autoplaced yes)
-		(property "Reference" "U3"
+		(property "Reference" "U2"
 			(at 163.83 45.72 0)
 			(effects
@@
 			(project "drum_trigger"
 				(path "/5aab9db2-4b7f-4c4d-b6d6-4c2a1995e627/7d7842c4-e5e3-46ac-bf06-c89ddb20aca8"
-					(reference "U3")
+					(reference "U2")
 					(unit 1)
 				)
@@
 		(on_board yes)
 		(dnp no)
-		(property "Reference" "C19"
+		(property "Reference" "C20"
 			(at 178.816 102.362 90)
 			(effects
@@
 			(project "drum_trigger"
 				(path "/5aab9db2-4b7f-4c4d-b6d6-4c2a1995e627/7d7842c4-e5e3-46ac-bf06-c89ddb20aca8"
-					(reference "C19")
+					(reference "C20")
 					(unit 1)
 				)
@@
 		(dnp no)
 		(fields_autoplaced yes)
-		(property "Reference" "#PWR040"
+		(property "Reference" "#PWR042"
 			(at 180.34 73.66 0)
 			(effects
@@
 			(project "drum_trigger"
 				(path "/5aab9db2-4b7f-4c4d-b6d6-4c2a1995e627/7d7842c4-e5e3-46ac-bf06-c89ddb20aca8"
-					(reference "#PWR040")
+					(reference "#PWR042")
 					(unit 1)
 				)
@@
 		(on_board yes)
 		(dnp no)
-		(property "Reference" "C16"
+		(property "Reference" "C17"
 			(at 144.526 57.912 90)
 			(effects
@@
 			(project "drum_trigger"
 				(path "/5aab9db2-4b7f-4c4d-b6d6-4c2a1995e627/7d7842c4-e5e3-46ac-bf06-c89ddb20aca8"
-					(reference "C16")
+					(reference "C17")
 					(unit 1)
 				)
